File: SevenSegmentClock/display.kicad_sch (KiCad schematic)
At the start: 104 parts, among them Q1 PN2222A, Q2 PN2222A, Q3 PN2222A, Q4 PN2222A, Q5 PN2222A, Q6 PN2222A, Q7 13N50F, U1 4511, U10 4042, U11 4511, U12 4511, U2 4504, U3 4511, U4 4042, U5 4511, U6 4504, U7 74HC138, U8 4511, U9 4082

Commit message: Fixing incorrect footprints
Parts:
- U1, U11, U12, U2, U3, U5, U6, U8: footprint Package_SO:SOIC-16W_5.3x10.2mm_P1.27mm -> Package_SO:SOIC-16_3.9x9.9mm_P1.27mm
Changed lines of the file:
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@@
     (property "Reference" "U1" (id 0) (at 141.986 27.1612 0))
     (property "Value" "4511" (id 1) (at 141.986 30.2061 0))
-    (property "Footprint" "Package_SO:SOIC-16W_5.3x10.2mm_P1.27mm" (id 2) (at 141.986 27.94 0)
+    (property "Footprint" "Package_SO:SOIC-16_3.9x9.9mm_P1.27mm" (id 2) (at 141.986 27.94 0)
       (effects (font (size 1.27 1.27)) hide)
     )
@@
       (effects (font (size 1.27 1.27)) (justify left))
     )
-    (property "Footprint" "Package_SO:SOIC-16W_5.3x10.2mm_P1.27mm" (id 2) (at 76.327 73.66 0)
+    (property "Footprint" "Package_SO:SOIC-16_3.9x9.9mm_P1.27mm" (id 2) (at 76.327 73.66 0)
       (effects (font (size 1.27 1.27)) hide)
     )
@@
     (property "Reference" "U8" (id 0) (at 141.986 145.2712 0))
     (property "Value" "4511" (id 1) (at 141.986 148.3161 0))
-    (property "Footprint" "Package_SO:SOIC-16W_5.3x10.2mm_P1.27mm" (id 2) (at 141.986 146.05 0)
+    (property "Footprint" "Package_SO:SOIC-16_3.9x9.9mm_P1.27mm" (id 2) (at 141.986 146.05 0)
       (effects (font (size 1.27 1.27)) hide)
     )
@@
     (property "Reference" "U5" (id 0) (at 141.986 114.7912 0))
     (property "Value" "4511" (id 1) (at 141.986 117.8361 0))
-    (property "Footprint" "Package_SO:SOIC-16W_5.3x10.2mm_P1.27mm" (id 2) (at 141.986 115.57 0)
+    (property "Footprint" "Package_SO:SOIC-16_3.9x9.9mm_P1.27mm" (id 2) (at 141.986 115.57 0)
       (effects (font (size 1.27 1.27)) hide)
     )
@@
     (property "Reference" "U3" (id 0) (at 141.986 58.9112 0))
     (property "Value" "4511" (id 1) (at 141.986 61.9561 0))
-    (property "Footprint" "Package_SO:SOIC-16W_5.3x10.2mm_P1.27mm" (id 2) (at 141.986 59.69 0)
+    (property "Footprint" "Package_SO:SOIC-16_3.9x9.9mm_P1.27mm" (id 2) (at 141.986 59.69 0)
       (effects (font (size 1.27 1.27)) hide)
     )
@@
     (property "Reference" "U11" (id 0) (at 141.986 200.3892 0))
     (property "Value" "4511" (id 1) (at 141.986 202.9261 0))
-    (property "Footprint" "Package_SO:SOIC-16W_5.3x10.2mm_P1.27mm" (id 2) (at 141.986 200.66 0)
+    (property "Footprint" "Package_SO:SOIC-16_3.9x9.9mm_P1.27mm" (id 2) (at 141.986 200.66 0)
       (effects (font (size 1.27 1.27)) hide)
     )
@@
       (effects (font (size 1.27 1.27)) (justify left))
     )
-    (property "Footprint" "Package_SO:SOIC-16W_5.3x10.2mm_P1.27mm" (id 2) (at 87.122 168.91 0)
+    (property "Footprint" "Package_SO:SOIC-16_3.9x9.9mm_P1.27mm" (id 2) (at 87.122 168.91 0)
       (effects (font (size 1.27 1.27)) hide)
     )
@@
     (property "Reference" "U12" (id 0) (at 141.986 229.8532 0))
     (property "Value" "4511" (id 1) (at 141.986 233.6093 0))
-    (property "Footprint" "Package_SO:SOIC-16W_5.3x10.2mm_P1.27mm" (id 2) (at 141.986 231.14 0)
-      (effects (font (size 1.27 1.27)) hide)
-    )
+    (property "Footprint" "Package_SO:SOIC-16_3.9x9.9mm_P1.27mm" (id 2) (at 141.986 231.14 0)
+      (effects (font (size 1.27 1.27)) hide)
+    )

Commit message: The 560R resistor was not available in a SMD package
Parts:
- R16, R19, R36, R39: footprint Resistor_SMD:R_1206_3216Metric_Pad1.30x1.75mm_HandSolder -> Resistor_THT:R_Axial_DIN0207_L6.3mm_D2.5mm_P10.16mm_Horizontal
Changed lines of the file:
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@@
       (effects (font (size 1.27 1.27)) (justify right))
     )
-    (property "Footprint" "Resistor_SMD:R_1206_3216Metric_Pad1.30x1.75mm_HandSolder" (id 2) (at 186.944 93.345 90)
+    (property "Footprint" "Resistor_THT:R_Axial_DIN0207_L6.3mm_D2.5mm_P10.16mm_Horizontal" (id 2) (at 186.944 93.345 90)
       (effects (font (size 1.27 1.27)) hide)
     )
@@
       (effects (font (size 1.27 1.27)) (justify right))
     )
-    (property "Footprint" "Resistor_SMD:R_1206_3216Metric_Pad1.30x1.75mm_HandSolder" (id 2) (at 184.404 83.185 90)
+    (property "Footprint" "Resistor_THT:R_Axial_DIN0207_L6.3mm_D2.5mm_P10.16mm_Horizontal" (id 2) (at 184.404 83.185 90)
       (effects (font (size 1.27 1.27)) hide)
     )
@@
       (effects (font (size 1.27 1.27)) (justify right))
     )
-    (property "Footprint" "Resistor_SMD:R_1206_3216Metric_Pad1.30x1.75mm_HandSolder" (id 2) (at 186.309 181.61 90)
+    (property "Footprint" "Resistor_THT:R_Axial_DIN0207_L6.3mm_D2.5mm_P10.16mm_Horizontal" (id 2) (at 186.309 181.61 90)
       (effects (font (size 1.27 1.27)) hide)
     )
@@
       (effects (font (size 1.27 1.27)) (justify right))
     )
-    (property "Footprint" "Resistor_SMD:R_1206_3216Metric_Pad1.30x1.75mm_HandSolder" (id 2) (at 184.404 170.18 90)
-      (effects (font (size 1.27 1.27)) hide)
-    )
+    (property "Footprint" "Resistor_THT:R_Axial_DIN0207_L6.3mm_D2.5mm_P10.16mm_Horizontal" (id 2) (at 184.404 170.18 90)
+      (effects (font (size 1.27 1.27)) hide)
+    )

Commit message: WIP: PCB Design
Connections:
- net at R18.1: now also U4.1; no longer U4.10
- net at R38.1: now also U4.10; no longer U4.1
Changed lines of the file:
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@@
+    (stroke (width 0) (type default) (color 0 0 0 0))
+  )
+  (wire (pts (xy 128.016 100.33) (xy 128.016 90.17))
     (stroke (width 0) (type default) (color 0 0 0 0))
   )
@@
     (stroke (width 0) (type default) (color 0 0 0 0))
   )
-  (wire (pts (xy 108.458 177.165) (xy 108.458 100.33))
+  (wire (pts (xy 108.458 90.17) (xy 108.458 177.165))
     (stroke (width 0) (type default) (color 0 0 0 0))
   )
@@
     (stroke (width 0) (type default) (color 0 0 0 0))
   )
+  (wire (pts (xy 101.092 90.17) (xy 108.458 90.17))
+    (stroke (width 0) (type default) (color 0 0 0 0))
+  )
   (wire (pts (xy 84.582 111.76) (xy 84.582 113.03))
     (stroke (width 0) (type default) (color 0 0 0 0))
@@
     (stroke (width 0) (type default) (color 0 0 0 0))
   )
-  (wire (pts (xy 101.092 90.17) (xy 129.286 90.17))
-    (stroke (width 0) (type default) (color 0 0 0 0))
-  )
   (wire (pts (xy 129.286 177.165) (xy 108.458 177.165))
     (stroke (width 0) (type default) (color 0 0 0 0))
@@
     (stroke (width 0) (type default) (color 0 0 0 0))
   )
+  (wire (pts (xy 101.092 100.33) (xy 128.016 100.33))
+    (stroke (width 0) (type default) (color 0 0 0 0))
+  )
   (wire (pts (xy 77.597 197.866) (xy 77.597 198.501))
     (stroke (width 0) (type default) (color 0 0 0 0))
@@
     (stroke (width 0) (type default) (color 0 0 0 0))
   )
-  (wire (pts (xy 101.092 100.33) (xy 108.458 100.33))
-    (stroke (width 0) (type default) (color 0 0 0 0))
-  )
   (wire (pts (xy 42.037 270.002) (xy 45.085 270.002))
     (stroke (width 0) (type default) (color 0 0 0 0))
@@
     (stroke (width 0) (type default) (color 0 0 0 0))
   )
+  (wire (pts (xy 128.016 90.17) (xy 129.286 90.17))
+    (stroke (width 0) (type default) (color 0 0 0 0))
+  )

Commit message: WIP: PCB design
Parts:
- C1, C10, C11, C12, C13, C14, C2, C3, C4, C5, C6, C7, C8, C9: footprint Capacitor_THT:C_Disc_D5.0mm_W2.5mm_P5.00mm -> Capacitor_SMD:C_1206_3216Metric_Pad1.33x1.80mm_HandSolder
Connections:
- net at R38.1: now also U4.11; no longer U4.10
- net at R35.1: now also U4.10; no longer U4.11
Changed lines of the file:
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@@
     (stroke (width 0) (type default) (color 0 0 0 0))
   )
-  (wire (pts (xy 101.092 95.25) (xy 109.855 95.25))
-    (stroke (width 0) (type default) (color 0 0 0 0))
-  )
   (wire (pts (xy 116.586 146.05) (xy 128.016 146.05))
     (stroke (width 0) (type default) (color 0 0 0 0))
@@
     (stroke (width 0) (type default) (color 0 0 0 0))
   )
+  (wire (pts (xy 108.458 95.25) (xy 108.458 177.165))
+    (stroke (width 0) (type default) (color 0 0 0 0))
+  )
   (wire (pts (xy 141.986 36.83) (xy 141.986 38.1))
     (stroke (width 0) (type default) (color 0 0 0 0))
@@
     (stroke (width 0) (type default) (color 0 0 0 0))
   )
-  (wire (pts (xy 108.458 90.17) (xy 108.458 177.165))
+  (wire (pts (xy 109.855 90.17) (xy 101.092 90.17))
     (stroke (width 0) (type default) (color 0 0 0 0))
   )
@@
     (stroke (width 0) (type default) (color 0 0 0 0))
   )
+  (wire (pts (xy 101.092 95.25) (xy 108.458 95.25))
+    (stroke (width 0) (type default) (color 0 0 0 0))
+  )
   (wire (pts (xy 190.246 140.97) (xy 195.326 140.97))
     (stroke (width 0) (type default) (color 0 0 0 0))
@@
     (stroke (width 0) (type default) (color 0 0 0 0))
   )
-  (wire (pts (xy 109.855 165.735) (xy 109.855 95.25))
+  (wire (pts (xy 109.855 90.17) (xy 109.855 165.735))
     (stroke (width 0) (type default) (color 0 0 0 0))
   )
@@
     (stroke (width 0) (type default) (color 0 0 0 0))
   )
-  (wire (pts (xy 101.092 90.17) (xy 108.458 90.17))
-    (stroke (width 0) (type default) (color 0 0 0 0))
-  )
   (wire (pts (xy 84.582 111.76) (xy 84.582 113.03))
     (stroke (width 0) (type default) (color 0 0 0 0))
@@
       (effects (font (size 1.27 1.27)) (justify left))
     )
-    (property "Footprint" "Capacitor_THT:C_Disc_D5.0mm_W2.5mm_P5.00mm" (id 2) (at 42.4942 260.223 0)
+    (property "Footprint" "Capacitor_SMD:C_1206_3216Metric_Pad1.33x1.80mm_HandSolder" (id 2) (at 42.4942 260.223 0)
       (effects (font (size 1.27 1.27)) hide)
     )
@@
       (effects (font (size 1.27 1.27)) (justify left))
     )
-    (property "Footprint" "Capacitor_THT:C_Disc_D5.0mm_W2.5mm_P5.00mm" (id 2) (at 39.4462 278.765 0)
+    (property "Footprint" "Capacitor_SMD:C_1206_3216Metric_Pad1.33x1.80mm_HandSolder" (id 2) (at 39.4462 278.765 0)
       (effects (font (size 1.27 1.27)) hide)
     )
@@
       (effects (font (size 1.27 1.27)) (justify left))
     )
-    (property "Footprint" "Capacitor_THT:C_Disc_D5.0mm_W2.5mm_P5.00mm" (id 2) (at 15.9512 260.223 0)
+    (property "Footprint" "Capacitor_SMD:C_1206_3216Metric_Pad1.33x1.80mm_HandSolder" (id 2) (at 15.9512 260.223 0)
       (effects (font (size 1.27 1.27)) hide)
     )
@@
       (effects (font (size 1.27 1.27)) (justify left))
     )
-    (property "Footprint" "Capacitor_THT:C_Disc_D5.0mm_W2.5mm_P5.00mm" (id 2) (at 59.3852 278.765 0)
+    (property "Footprint" "Capacitor_SMD:C_1206_3216Metric_Pad1.33x1.80mm_HandSolder" (id 2) (at 59.3852 278.765 0)
       (effects (font (size 1.27 1.27)) hide)
     )
@@
       (effects (font (size 1.27 1.27)) (justify left))
     )
-    (property "Footprint" "Capacitor_THT:C_Disc_D5.0mm_W2.5mm_P5.00mm" (id 2) (at 19.1262 278.765 0)
+    (property "Footprint" "Capacitor_SMD:C_1206_3216Metric_Pad1.33x1.80mm_HandSolder" (id 2) (at 19.1262 278.765 0)
       (effects (font (size 1.27 1.27)) hide)
     )
@@
       (effects (font (size 1.27 1.27)) (justify left))
     )
-    (property "Footprint" "Capacitor_THT:C_Disc_D5.0mm_W2.5mm_P5.00mm" (id 2) (at 32.8422 278.765 0)
+    (property "Footprint" "Capacitor_SMD:C_1206_3216Metric_Pad1.33x1.80mm_HandSolder" (id 2) (at 32.8422 278.765 0)
       (effects (font (size 1.27 1.27)) hide)
     )
@@
       (effects (font (size 1.27 1.27)) (justify left))
     )
-    (property "Footprint" "Capacitor_THT:C_Disc_D5.0mm_W2.5mm_P5.00mm" (id 2) (at 52.6542 278.765 0)
+    (property "Footprint" "Capacitor_SMD:C_1206_3216Metric_Pad1.33x1.80mm_HandSolder" (id 2) (at 52.6542 278.765 0)
       (effects (font (size 1.27 1.27)) hide)
     )
@@
       (effects (font (size 1.27 1.27)) (justify left))
     )
-    (property "Footprint" "Capacitor_THT:C_Disc_D5.0mm_W2.5mm_P5.00mm" (id 2) (at 29.1592 260.223 0)
+    (property "Footprint" "Capacitor_SMD:C_1206_3216Metric_Pad1.33x1.80mm_HandSolder" (id 2) (at 29.1592 260.223 0)
       (effects (font (size 1.27 1.27)) hide)
     )
@@
       (effects (font (size 1.27 1.27)) (justify left))
     )
-    (property "Footprint" "Capacitor_THT:C_Disc_D5.0mm_W2.5mm_P5.00mm" (id 2) (at 46.0502 278.765 0)
+    (property "Footprint" "Capacitor_SMD:C_1206_3216Metric_Pad1.33x1.80mm_HandSolder" (id 2) (at 46.0502 278.765 0)
       (effects (font (size 1.27 1.27)) hide)
     )
@@
       (effects (font (size 1.27 1.27)) (justify left))
     )
-    (property "Footprint" "Capacitor_THT:C_Disc_D5.0mm_W2.5mm_P5.00mm" (id 2) (at 35.6362 260.223 0)
+    (property "Footprint" "Capacitor_SMD:C_1206_3216Metric_Pad1.33x1.80mm_HandSolder" (id 2) (at 35.6362 260.223 0)
       (effects (font (size 1.27 1.27)) hide)
     )
@@
       (effects (font (size 1.27 1.27)) (justify left))
     )
-    (property "Footprint" "Capacitor_THT:C_Disc_D5.0mm_W2.5mm_P5.00mm" (id 2) (at 25.8572 278.765 0)
+    (property "Footprint" "Capacitor_SMD:C_1206_3216Metric_Pad1.33x1.80mm_HandSolder" (id 2) (at 25.8572 278.765 0)
       (effects (font (size 1.27 1.27)) hide)
     )
@@
       (effects (font (size 1.27 1.27)) (justify left))
     )
-    (property "Footprint" "Capacitor_THT:C_Disc_D5.0mm_W2.5mm_P5.00mm" (id 2) (at 66.1162 278.765 0)
+    (property "Footprint" "Capacitor_SMD:C_1206_3216Metric_Pad1.33x1.80mm_HandSolder" (id 2) (at 66.1162 278.765 0)
       (effects (font (size 1.27 1.27)) hide)
     )
@@
       (effects (font (size 1.27 1.27)) (justify left))
     )
-    (property "Footprint" "Capacitor_THT:C_Disc_D5.0mm_W2.5mm_P5.00mm" (id 2) (at 22.5552 260.223 0)
+    (property "Footprint" "Capacitor_SMD:C_1206_3216Metric_Pad1.33x1.80mm_HandSolder" (id 2) (at 22.5552 260.223 0)
       (effects (font (size 1.27 1.27)) hide)
     )
@@
       (effects (font (size 1.27 1.27)) (justify left))
     )
-    (property "Footprint" "Capacitor_THT:C_Disc_D5.0mm_W2.5mm_P5.00mm" (id 2) (at 49.7332 260.223 0)
+    (property "Footprint" "Capacitor_SMD:C_1206_3216Metric_Pad1.33x1.80mm_HandSolder" (id 2) (at 49.7332 260.223 0)
       (effects (font (size 1.27 1.27)) hide)
     )
