File: SevenSegmentClock/SevenSegmentClock.kicad_pcb (KiCad board)
At the start: 2 copper layers, 87 parts, among them Q1 PN2222A, Q2 PN2222A, Q3 PN2222A, Q4 PN2222A, U1 4504, U10 4511, U11 ESP8266, U2 74LS138, U3 4504, U4 4042, U5 4511, U6 4511, U7 4511, U8 4511, U9 4511

Commit message: Fixing incorrect footprints
Parts:
- added C13: 100nF, Capacitor_THT:C_Disc_D5.0mm_W2.5mm_P5.00mm, F.Cu at (186.9, 97.5)
- added C14: 100nF, Capacitor_THT:C_Disc_D5.0mm_W2.5mm_P5.00mm, F.Cu at (186.9, 101.4)
- added C15: 4.7uF, Capacitor_THT:CP_Radial_D6.3mm_P2.50mm, F.Cu at (204.9, 111.6)
- added C16: 100nF, Capacitor_THT:C_Disc_D5.0mm_W2.5mm_P5.00mm, F.Cu at (186.7, 109.4)
- added C17: 100nF, Capacitor_THT:C_Disc_D5.0mm_W2.5mm_P5.00mm, F.Cu at (186.7, 105.6)
- added C18: 47uF, Capacitor_THT:CP_Radial_D6.3mm_P2.50mm, F.Cu at (205.1, 97.0)
- added C19: 100nF, Capacitor_THT:C_Disc_D6.0mm_W2.5mm_P5.00mm, F.Cu at (186.6, 113.9)
- added C20: 47uF, Capacitor_THT:CP_Radial_D6.3mm_P2.50mm, F.Cu at (225.0, 96.6)
- added C21: 4.7uF, Capacitor_THT:CP_Radial_D6.3mm_P2.50mm, F.Cu at (224.8, 111.5)
- added C22: 100nF, Capacitor_THT:C_Disc_D6.0mm_W2.5mm_P5.00mm, F.Cu at (186.5, 117.7)
- added C23: 4.7uF, Capacitor_THT:CP_Radial_D6.3mm_P2.50mm, F.Cu at (233.4, 111.7)
- added C24: 47uF, Capacitor_THT:CP_Radial_D6.3mm_P2.50mm, F.Cu at (214.9, 96.7)
- added C25: 4.7uF, Capacitor_THT:CP_Radial_D6.3mm_P2.50mm, F.Cu at (214.4, 111.6)
- added C26: 470uF, Capacitor_THT:CP_Radial_D10.0mm_P5.00mm, F.Cu at (254.5, 104.3)
- added C27: 470uF, Capacitor_THT:CP_Radial_D10.0mm_P5.00mm, F.Cu at (270.1, 103.8)
- added J1: 12V, Connector_PinHeader_2.54mm:PinHeader_1x01_P2.54mm_Vertical, F.Cu at (169.3, 137.7)
- added J2: GND, Connector_PinHeader_2.54mm:PinHeader_1x01_P2.54mm_Vertical, F.Cu at (173.4, 137.3)
- added Q5: PN2222A, Package_TO_SOT_THT:TO-92_Inline, F.Cu at (78.5, 182.9)
- added Q6: PN2222A, Package_TO_SOT_THT:TO-92_Inline, F.Cu at (106.9, 182.6)
- added Q7: 13N50F, Package_TO_SOT_THT:TO-220-3_Vertical, F.Cu at (95.7, 194.6)
- added R51: 160R, Resistor_SMD:R_1206_3216Metric_Pad1.30x1.75mm_HandSolder, F.Cu at (218.9, 20.8)
- added R52: 160R, Resistor_SMD:R_1206_3216Metric_Pad1.30x1.75mm_HandSolder, F.Cu at (219.1, 16.8)
- added R53: 1k, Resistor_SMD:R_1206_3216Metric_Pad1.30x1.75mm_HandSolder, F.Cu at (198.7, 41.5)
- added R54: 160R, Resistor_SMD:R_1206_3216Metric_Pad1.30x1.75mm_HandSolder, F.Cu at (213.1, 32.4)
- added R55: 160R, Resistor_SMD:R_1206_3216Metric_Pad1.30x1.75mm_HandSolder, F.Cu at (213.1, 29.1)
- added R56: 160R, Resistor_SMD:R_1206_3216Metric_Pad1.30x1.75mm_HandSolder, F.Cu at (218.8, 25.1)
- added R57: 160R, Resistor_SMD:R_1206_3216Metric_Pad1.30x1.75mm_HandSolder, F.Cu at (218.7, 29.0)
- added R58: 1k, Resistor_SMD:R_1206_3216Metric_Pad1.30x1.75mm_HandSolder, F.Cu at (205.2, 41.4)
- added R59: 10k, Resistor_THT:R_Axial_DIN0207_L6.3mm_D2.5mm_P10.16mm_Horizontal, F.Cu at (196.1, 58.7)
- added R60: R_Photo, OptoDevice:R_LDR_4.9x4.2mm_P2.54mm_Vertical, F.Cu at (248.0, 77.2)
- added R61: 2.2M, Resistor_THT:R_Axial_DIN0207_L6.3mm_D2.5mm_P10.16mm_Horizontal, F.Cu at (169.7, 70.5)
- added R62: 1k, Resistor_SMD:R_1206_3216Metric_Pad1.30x1.75mm_HandSolder, F.Cu at (193.5, 41.5)
- added SSD7: HOU_TENS, Library:LSD230A, F.Cu at (40.0, 51.6)
- added SSD8: Percent, Display_7Segment:7SegmentLED_LTS6760_LTS6780, F.Cu at (30.2, 182.2)
- added U12: 4511, Package_SO:SOIC-16_3.9x9.9mm_P1.27mm, F.Cu at (87.5, 190.9)
- added U13: ESP8266, Library:ESP8266 (NodeMCU_12-E), F.Cu at (259.6, 42.8)
- added U14: DHT11, Sensor:Aosong_DHT11_5.5x12.0_P2.54mm, F.Cu at (261.5, 77.4)
- added U15: LM2596, Library:LM2596, F.Cu at (145.1, 177.9)
- R1, R2, R3, R4: value 1k -> 160R; footprint Resistor_THT:R_Axial_DIN0207_L6.3mm_D2.5mm_P7.62mm_Horizontal -> Resistor_SMD:R_1206_3216Metric_Pad1.30x1.75mm_HandSolder
- R10, R11, R12, R13, R14, R21, R22, R23, R24, R25, R26, R27, R28, R29, R30, R31, R32, R33, R34, R41, R42, R43, R44, R45, R46, R5, R6, R7, R8, R9: value 180R -> 160R; footprint Resistor_THT:R_Axial_DIN0207_L6.3mm_D2.5mm_P7.62mm_Horizontal -> Resistor_SMD:R_1206_3216Metric_Pad1.30x1.75mm_HandSolder
- R15, R18, R35, R38: value 180R -> 1k; footprint Resistor_THT:R_Axial_DIN0207_L6.3mm_D2.5mm_P7.62mm_Horizontal -> Resistor_SMD:R_1206_3216Metric_Pad1.30x1.75mm_HandSolder
- R16, R19, R36, R39: value 180R -> 560R; footprint Resistor_THT:R_Axial_DIN0207_L6.3mm_D2.5mm_P7.62mm_Horizontal -> Resistor_SMD:R_1206_3216Metric_Pad1.30x1.75mm_HandSolder
- R17, R20, R37, R40: value 180R -> 10k; footprint Resistor_THT:R_Axial_DIN0207_L6.3mm_D2.5mm_P7.62mm_Horizontal -> Resistor_THT:R_Axial_DIN0207_L6.3mm_D2.5mm_P10.16mm_Horizontal
- R47, R48, R49, R50: value 300R -> 160R; footprint Resistor_THT:R_Axial_DIN0207_L6.3mm_D2.5mm_P7.62mm_Horizontal -> Resistor_SMD:R_1206_3216Metric_Pad1.30x1.75mm_HandSolder
- SSD1: value LSD230A -> SEC_UNITS
- SSD2: value LSD230A -> SEC_TENS
- SSD3: value LSD230A -> MIN_UNITS
- SSD4: value LSD230A -> MIN_TENS
- SSD5: value LSD230A -> HOU_UNITS
- SSD6: value LSD230A -> Degree; footprint Library:LSD230A -> Display_7Segment:7SegmentLED_LTS6760_LTS6780
- U1, U3: value 4504 -> 4511
- U10: value 4511 -> 4042; footprint Package_SO:SOIC-16_3.9x9.9mm_P1.27mm -> Package_DIP:DIP-16_W7.62mm_Socket_LongPads
- U11: value ESP8266 -> 4511; footprint ESP8266:NodeMCU1.0(12-E) -> Package_SO:SOIC-16_3.9x9.9mm_P1.27mm
- U2: value 74LS138 -> 4504
- U4: footprint Package_DIP:DIP-16_W7.62mm_LongPads -> Package_DIP:DIP-16_W7.62mm_Socket_LongPads
- U5: moved to F.Cu
- U6: value 4511 -> 4504
- U7: value 4511 -> 74HC138
- U9: value 4511 -> 4082; footprint Package_SO:SOIC-16_3.9x9.9mm_P1.27mm -> Package_DIP:DIP-14_W7.62mm_Socket_LongPads
- moved U3 216.6 mm to (77.9, 191.0)
- moved U1 206.8 mm to (68.6, 191.0)
- moved U11 202.3 mm to (58.4, 191.0)
- moved U4 185.6 mm to (59.0, 164.0)
- moved U2 184.1 mm to (83.1, 167.1)
- moved Q2 136.8 mm to (84.2, 182.7)
- moved Q4 136.4 mm to (95.5, 182.8)
- moved U8 135.9 mm to (48.9, 191.0)
- moved Q3 135.7 mm to (90.0, 182.7)
- moved Q1 134.1 mm to (101.3, 182.7)
- moved SSD6 133.0 mm to (15.8, 182.2), turned to 90 degrees
- moved U9 131.9 mm to (15.8, 194.7), turned to 90 degrees
- moved D4 125.9 mm to (80.1, 177.8)
- moved D3 124.0 mm to (87.0, 177.8)
- moved U10 104.6 mm to (47.8, 164.4)
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Connections:
- C1 pad 1: +12V -> +3.3V
- C2 pad 1: +12V -> +3.3V
- C3 pad 1: +12V -> +3.3V
- C4 pad 1: +12V -> +3.3V
- C5 pad 1: +12V -> +3.3V
- C6 pad 1: +12V -> +3.3V
- Q1 pad 1: GND -> /Display/LedsGnd
- Q2 pad 1: GND -> /Display/LedsGnd
- Q3 pad 1: GND -> /Display/LedsGnd
- Q4 pad 1: GND -> /Display/LedsGnd
- R1 pad 2: Net-(Q1-Pad2) -> Net-(R1-Pad2)
- R15 pad 2: Net-(R15-Pad2) -> Net-(Q1-Pad2)
- R16 pad 1: Net-(R16-Pad1) -> Net-(D1-Pad2)
- R16 pad 2: Net-(R16-Pad2) -> +12V
- R17 pad 1: Net-(R17-Pad1) -> +12V
- R17 pad 2: Net-(R17-Pad2) -> Net-(D1-Pad1)
- R18 pad 2: Net-(R18-Pad2) -> Net-(Q2-Pad2)
- R19 pad 1: Net-(R19-Pad1) -> Net-(D2-Pad2)
- R19 pad 2: Net-(R19-Pad2) -> +12V
- R2 pad 2: Net-(Q2-Pad2) -> Net-(R2-Pad2)
- R20 pad 1: Net-(R20-Pad1) -> +12V
- R20 pad 2: Net-(R20-Pad2) -> Net-(D2-Pad1)
- R3 pad 2: Net-(Q3-Pad2) -> Net-(R3-Pad2)
- R35 pad 2: Net-(R35-Pad2) -> Net-(Q3-Pad2)
- R36 pad 1: Net-(R36-Pad1) -> Net-(D3-Pad2)
- R36 pad 2: Net-(R36-Pad2) -> +12V
- R37 pad 1: Net-(R37-Pad1) -> +12V
- R37 pad 2: Net-(R37-Pad2) -> Net-(D3-Pad1)
- R38 pad 2: Net-(R38-Pad2) -> Net-(Q4-Pad2)
- R39 pad 1: Net-(R39-Pad1) -> Net-(D4-Pad2)
- R39 pad 2: Net-(R39-Pad2) -> +12V
- R4 pad 2: Net-(Q4-Pad2) -> Net-(R4-Pad2)
- R40 pad 1: Net-(R40-Pad1) -> +12V
- R40 pad 2: Net-(R40-Pad2) -> Net-(D4-Pad1)
- R47 pad 1: Net-(D1-Pad2) -> Net-(R47-Pad1)
- R47 pad 2: +12V -> Net-(R47-Pad2)
- R48 pad 1: Net-(D3-Pad2) -> Net-(R48-Pad1)
- R48 pad 2: +12V -> Net-(R48-Pad2)
- R49 pad 1: Net-(D4-Pad2) -> Net-(R49-Pad1)
- R49 pad 2: +12V -> Net-(R49-Pad2)
- R50 pad 1: Net-(D2-Pad2) -> Net-(Q5-Pad3)
- R50 pad 2: +12V -> Net-(R50-Pad2)
- SSD1 pad 10: Net-(R11-Pad2) -> Net-(R7-Pad2)
- SSD1 pad 2: Net-(R9-Pad2) -> Net-(R5-Pad2)
- SSD1 pad 3: Net-(R8-Pad2) -> Net-(R4-Pad2)
- SSD1 pad 4: Net-(R7-Pad2) -> Net-(R3-Pad2)
- SSD1 pad 6: Net-(R6-Pad2) -> Net-(R2-Pad2)
- SSD1 pad 7: Net-(R5-Pad2) -> Net-(R1-Pad2)
- SSD1 pad 9: Net-(R10-Pad2) -> Net-(R6-Pad2)
- SSD2 pad 10: Net-(R18-Pad2) -> Net-(R14-Pad2)
- SSD2 pad 2: Net-(R16-Pad2) -> Net-(R12-Pad2)
- SSD2 pad 3: Net-(R15-Pad2) -> Net-(R11-Pad2)
- SSD2 pad 4: Net-(R14-Pad2) -> Net-(R10-Pad2)
- SSD2 pad 6: Net-(R13-Pad2) -> Net-(R9-Pad2)
- SSD2 pad 7: Net-(R12-Pad2) -> Net-(R8-Pad2)
- SSD2 pad 9: Net-(R17-Pad2) -> Net-(R13-Pad2)
- SSD3 pad 10: Net-(R25-Pad2) -> Net-(R27-Pad2)
- SSD3 pad 2: Net-(R23-Pad2) -> Net-(R25-Pad2)
- SSD3 pad 3: Net-(R22-Pad2) -> Net-(R24-Pad2)
- SSD3 pad 4: Net-(R21-Pad2) -> Net-(R23-Pad2)
- SSD3 pad 6: Net-(R20-Pad2) -> Net-(R22-Pad2)
- SSD3 pad 7: Net-(R19-Pad2) -> Net-(R21-Pad2)
- SSD3 pad 9: Net-(R24-Pad2) -> Net-(R26-Pad2)
- SSD4 pad 10: Net-(R32-Pad2) -> Net-(R34-Pad2)
- SSD4 pad 2: Net-(R30-Pad2) -> Net-(R32-Pad2)
- SSD4 pad 3: Net-(R29-Pad2) -> Net-(R31-Pad2)
- SSD4 pad 4: Net-(R28-Pad2) -> Net-(R30-Pad2)
- SSD4 pad 6: Net-(R27-Pad2) -> Net-(R29-Pad2)
- SSD4 pad 7: Net-(R26-Pad2) -> Net-(R28-Pad2)
- SSD4 pad 9: Net-(R31-Pad2) -> Net-(R33-Pad2)
- SSD5 pad 10: Net-(R39-Pad2) -> Net-(R47-Pad2)
- SSD5 pad 2: Net-(R37-Pad2) -> Net-(R45-Pad2)
- SSD5 pad 3: Net-(R36-Pad2) -> Net-(R44-Pad2)
- SSD5 pad 4: Net-(R35-Pad2) -> Net-(R43-Pad2)
- SSD5 pad 6: Net-(R34-Pad2) -> Net-(R42-Pad2)
- SSD5 pad 7: Net-(R33-Pad2) -> Net-(R41-Pad2)
- SSD5 pad 9: Net-(R38-Pad2) -> Net-(R46-Pad2)
- SSD6 pad 1: GND -> +12V
- SSD6 pad 10: Net-(R46-Pad2) -> Net-(R50-Pad2)
- SSD6 pad 2: Net-(R44-Pad2) -> +12V
- SSD6 pad 3: Net-(R43-Pad2) -> +12V
- SSD6 pad 4: Net-(R42-Pad2) -> +12V
- SSD6 pad 5: GND -> +12V
- SSD6 pad 6: Net-(R41-Pad2) -> Net-(R50-Pad2)
- SSD6 pad 7: Net-(R40-Pad2) -> Net-(R50-Pad2)
- SSD6 pad 8: GND -> +12V
- SSD6 pad 9: Net-(R45-Pad2) -> Net-(R50-Pad2)
- U1 pad 1: +12V -> Net-(U1-Pad1)
- U1 pad 10: Net-(U1-Pad10) -> Net-(R4-Pad1)
- U1 pad 11: ~{BlkDisp} -> Net-(R3-Pad1)
- U1 pad 12: Net-(U1-Pad12) -> Net-(R2-Pad1)
- U1 pad 13: GND -> Net-(R1-Pad1)
- U1 pad 14: GND -> Net-(R7-Pad1)
- U1 pad 15: unconnected-(U1-Pad15) -> Net-(R6-Pad1)
- U1 pad 3: DispA -> +12V
- U1 pad 4: Net-(U1-Pad4) -> /Display/~{BlkDispBuf}
- U1 pad 5: DispB -> Net-(U1-Pad5)
- U1 pad 7: DispC -> Net-(U1-Pad7)
- U1 pad 9: DispD -> Net-(R5-Pad1)
- U10 pad 1: Net-(U1-Pad4) -> Net-(U10-Pad1)
- U10 pad 10: Net-(R43-Pad1) -> Net-(U10-Pad10)
- U10 pad 11: Net-(R42-Pad1) -> Net-(U10-Pad11)
- U10 pad 12: Net-(R41-Pad1) -> unconnected-(U10-Pad12)
- U10 pad 13: Net-(R40-Pad1) -> DispC
- U10 pad 14: Net-(R46-Pad1) -> DispD
- U10 pad 15: Net-(R45-Pad1) -> unconnected-(U10-Pad15)
- U10 pad 16: +12V -> +3.3V
- U10 pad 2: Net-(U1-Pad6) -> Net-(U10-Pad2)
- U10 pad 3: +12V -> unconnected-(U10-Pad3)
- U10 pad 4: Net-(U1-Pad12) -> DispA
- U10 pad 6: Net-(U1-Pad10) -> +3.3V
- U10 pad 7: Net-(U1-Pad2) -> DispB
- U10 pad 9: Net-(R44-Pad1) -> unconnected-(U10-Pad9)
- U11 pad 1: unconnected-(U11-Pad1) -> Net-(U1-Pad1)
- U11 pad 10: unconnected-(U11-Pad10) -> Net-(R44-Pad1)
- U11 pad 11: unconnected-(U11-Pad11) -> Net-(R43-Pad1)
- U11 pad 12: unconnected-(U11-Pad12) -> Net-(R42-Pad1)
- U11 pad 13: unconnected-(U11-Pad13) -> Net-(R41-Pad1)
- U11 pad 14: unconnected-(U11-Pad14) -> Net-(R47-Pad1)
- U11 pad 15: unconnected-(U11-Pad15) -> Net-(R46-Pad1)
- U11 pad 16: unconnected-(U11-Pad16) -> +12V
- U11 pad 2: unconnected-(U11-Pad2) -> Net-(U1-Pad2)
- U11 pad 3: unconnected-(U11-Pad3) -> +12V
- U11 pad 4: unconnected-(U11-Pad4) -> /Display/~{BlkDispBuf}
- U11 pad 5: unconnected-(U11-Pad5) -> Net-(U11-Pad5)
- U11 pad 6: unconnected-(U11-Pad6) -> Net-(U1-Pad6)
- U11 pad 7: unconnected-(U11-Pad7) -> Net-(U1-Pad7)
- U11 pad 8: unconnected-(U11-Pad8) -> GND
- U11 pad 9: unconnected-(U11-Pad9) -> Net-(R45-Pad1)
- U2 pad 1: DispSel0 -> +3.3V
- U2 pad 10: Net-(U2-Pad10) -> Net-(U1-Pad6)
- U2 pad 11: Net-(U2-Pad11) -> ~{BlkDisp}
- U2 pad 12: Net-(U2-Pad12) -> /Display/~{BlkDispBuf}
- U2 pad 13: Net-(U2-Pad13) -> GND
- U2 pad 14: Net-(U2-Pad14) -> GND
- U2 pad 15: Net-(U2-Pad15) -> unconnected-(U2-Pad15)
- U2 pad 2: DispSel1 -> Net-(U1-Pad7)
- U2 pad 3: DispSel2 -> DispA
- U2 pad 4: GND -> Net-(U1-Pad1)
- U2 pad 5: GND -> DispB
- U2 pad 6: +12V -> Net-(U1-Pad2)
- U2 pad 7: unconnected-(U2-Pad7) -> DispC
- U2 pad 9: /Display/DotsClk -> DispD
- U3 pad 1: +12V -> Net-(U1-Pad1)
- U3 pad 10: Net-(U3-Pad10) -> Net-(R11-Pad1)
- U3 pad 11: Net-(U2-Pad11) -> Net-(R10-Pad1)
- U3 pad 12: Net-(U3-Pad12) -> Net-(R9-Pad1)
- U3 pad 13: GND -> Net-(R8-Pad1)
- U3 pad 14: Net-(U2-Pad10) -> Net-(R14-Pad1)
- U3 pad 15: Net-(U10-Pad5) -> Net-(R13-Pad1)
- U3 pad 2: Net-(U3-Pad2) -> Net-(U1-Pad2)
- U3 pad 3: Net-(U2-Pad15) -> +12V
- U3 pad 4: Net-(U3-Pad4) -> /Display/~{BlkDispBuf}
- U3 pad 5: Net-(U2-Pad14) -> Net-(U3-Pad5)
- U3 pad 6: Net-(U3-Pad6) -> Net-(U1-Pad6)
- U3 pad 7: Net-(U2-Pad13) -> Net-(U1-Pad7)
- U3 pad 9: Net-(U2-Pad12) -> Net-(R12-Pad1)
- U4 pad 1: Net-(R4-Pad1) -> Net-(R38-Pad1)
- U4 pad 10: Net-(R2-Pad1) -> Net-(R18-Pad1)
- U4 pad 11: Net-(R3-Pad1) -> Net-(R35-Pad1)
- U4 pad 14: ~{BlkDisp} -> DispD
- U4 pad 16: +12V -> +3.3V
- U4 pad 2: Net-(R1-Pad1) -> Net-(R15-Pad1)
- U4 pad 6: +12V -> +3.3V
- U5 pad 1: Net-(U1-Pad4) -> Net-(U1-Pad1)
- U5 pad 10: Net-(R8-Pad1) -> Net-(R24-Pad1)
- U5 pad 11: Net-(R7-Pad1) -> Net-(R23-Pad1)
- U5 pad 12: Net-(R6-Pad1) -> Net-(R22-Pad1)
- U5 pad 13: Net-(R5-Pad1) -> Net-(R21-Pad1)
- U5 pad 14: Net-(R11-Pad1) -> Net-(R27-Pad1)
- U5 pad 15: Net-(R10-Pad1) -> Net-(R26-Pad1)
- U5 pad 2: Net-(U1-Pad6) -> Net-(U1-Pad2)
- U5 pad 4: Net-(U1-Pad12) -> /Display/~{BlkDispBuf}
- U5 pad 5: Net-(U3-Pad2) -> Net-(U5-Pad5)
- U5 pad 6: Net-(U1-Pad10) -> Net-(U1-Pad6)
- U5 pad 7: Net-(U1-Pad2) -> Net-(U1-Pad7)
- U5 pad 9: Net-(R9-Pad1) -> Net-(R25-Pad1)
- U6 pad 1: Net-(U1-Pad4) -> +3.3V
- U6 pad 10: Net-(R15-Pad1) -> Net-(U6-Pad10)
- U6 pad 11: Net-(R14-Pad1) -> Net-(U6-Pad11)
- U6 pad 12: Net-(R13-Pad1) -> Net-(U11-Pad5)
- U6 pad 13: Net-(R12-Pad1) -> GND
- U6 pad 14: Net-(R18-Pad1) -> Net-(U10-Pad5)
- U6 pad 15: Net-(R17-Pad1) -> Net-(U12-Pad5)
- U6 pad 2: Net-(U1-Pad6) -> Net-(U1-Pad5)
- U6 pad 3: +12V -> Net-(U6-Pad3)
- U6 pad 4: Net-(U1-Pad12) -> Net-(U3-Pad5)
- U6 pad 5: Net-(U3-Pad4) -> Net-(U6-Pad5)
- U6 pad 6: Net-(U1-Pad10) -> Net-(U5-Pad5)
- U6 pad 7: Net-(U1-Pad2) -> Net-(U6-Pad7)
- U6 pad 9: Net-(R16-Pad1) -> Net-(U6-Pad9)
- U7 pad 1: Net-(U1-Pad4) -> DispSel0
- U7 pad 10: Net-(R22-Pad1) -> Net-(U10-Pad5)
- U7 pad 11: Net-(R21-Pad1) -> Net-(U6-Pad11)
- U7 pad 12: Net-(R20-Pad1) -> Net-(U6-Pad9)
- U7 pad 13: Net-(R19-Pad1) -> Net-(U6-Pad7)
- U7 pad 14: Net-(R25-Pad1) -> Net-(U6-Pad5)
- U7 pad 15: Net-(R24-Pad1) -> Net-(U6-Pad3)
- U7 pad 16: +12V -> +3.3V
- U7 pad 2: Net-(U1-Pad6) -> DispSel1
- U7 pad 3: +12V -> DispSel2
- U7 pad 4: Net-(U1-Pad12) -> GND
- U7 pad 5: Net-(U3-Pad6) -> GND
- U7 pad 6: Net-(U1-Pad10) -> +3.3V
- U7 pad 7: Net-(U1-Pad2) -> unconnected-(U7-Pad7)
- U7 pad 9: Net-(R23-Pad1) -> /Display/DotsClk
- U8 pad 1: Net-(U1-Pad4) -> Net-(U1-Pad1)
- U8 pad 10: Net-(R29-Pad1) -> Net-(R31-Pad1)
- U8 pad 11: Net-(R28-Pad1) -> Net-(R30-Pad1)
- U8 pad 12: Net-(R27-Pad1) -> Net-(R29-Pad1)
- U8 pad 13: Net-(R26-Pad1) -> Net-(R28-Pad1)
- U8 pad 14: Net-(R32-Pad1) -> Net-(R34-Pad1)
- U8 pad 15: Net-(R31-Pad1) -> Net-(R33-Pad1)
- U8 pad 2: Net-(U1-Pad6) -> Net-(U1-Pad2)
- U8 pad 4: Net-(U1-Pad12) -> /Display/~{BlkDispBuf}
- U8 pad 5: Net-(U3-Pad10) -> Net-(U6-Pad10)
- U8 pad 6: Net-(U1-Pad10) -> Net-(U1-Pad6)
- U8 pad 7: Net-(U1-Pad2) -> Net-(U1-Pad7)
- U8 pad 9: Net-(R30-Pad1) -> Net-(R32-Pad1)
- U9 pad 1: Net-(U1-Pad4) -> /Display/DispDegree
- U9 pad 10: Net-(R36-Pad1) -> Net-(U10-Pad1)
- U9 pad 11: Net-(R35-Pad1) -> Net-(U10-Pad11)
- U9 pad 12: Net-(R34-Pad1) -> Net-(U10-Pad10)
- U9 pad 13: Net-(R33-Pad1) -> /Display/DispPercent
- U9 pad 14: Net-(R39-Pad1) -> +3.3V
- U9 pad 2: Net-(U1-Pad6) -> Net-(U10-Pad2)
- U9 pad 3: +12V -> Net-(U10-Pad10)
- U9 pad 4: Net-(U1-Pad12) -> Net-(U10-Pad11)
- U9 pad 5: Net-(U3-Pad12) -> Net-(U10-Pad1)
- U9 pad 6: Net-(U1-Pad10) -> unconnected-(U9-Pad6)
- U9 pad 7: Net-(U1-Pad2) -> GND
- U9 pad 8: GND -> unconnected-(U9-Pad8)
- U9 pad 9: Net-(R37-Pad1) -> +3.3V

Commit message: The 560R resistor was not available in a SMD package
Parts:
- R16, R19, R36, R39: footprint Resistor_SMD:R_1206_3216Metric_Pad1.30x1.75mm_HandSolder -> Resistor_THT:R_Axial_DIN0207_L6.3mm_D2.5mm_P10.16mm_Horizontal
- moved R16 16.7 mm to (171.2, 51.6)
- moved R36 7.62 mm to (184.2, 48.1)
- moved R39 4.02 mm to (184.3, 51.3)

Commit message: WIP: PCB Design
Parts:
- D1, D2, D3, D4, SSD1, SSD2, SSD3, SSD4, SSD5, SSD6, SSD7, SSD8: moved to B.Cu
- moved C16 338.3 mm to (514.4, 193.4)
- moved C20 338.3 mm to (552.7, 180.7)
- moved C26 338.3 mm to (582.1, 188.4)
- moved R59 338.3 mm to (523.7, 142.8)
- moved C18 338.3 mm to (532.8, 181.1)
- moved C2 338.3 mm to (505.5, 189.8)
- moved C24 338.3 mm to (542.5, 180.8)
- moved C27 338.3 mm to (597.8, 187.9)
- moved J2 338.3 mm to (501.0, 221.4)
- moved Q7 338.3 mm to (423.4, 278.7)
- moved R53 338.3 mm to (526.4, 125.5)
- moved R62 338.3 mm to (521.1, 125.6)
- moved C12 338.3 mm to (506.2, 193.8)
- moved C15 338.3 mm to (532.5, 195.7)
- moved C17 338.3 mm to (514.4, 189.6)
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Connections:
- R18 pad 1: Net-(R18-Pad1) -> Net-(U4-Pad1)
- U4 pad 1: Net-(R38-Pad1) -> Net-(U4-Pad1)
- U4 pad 10: Net-(R18-Pad1) -> Net-(R38-Pad1)
Routing:
- net +12V: track 0.00 -> 421.0 mm, vias 0 -> 10
- net Net-(U1-Pad6): track 0.00 -> 306.5 mm, vias 0 -> 7
- net Net-(U1-Pad7): track 0.00 -> 306.1 mm, vias 0 -> 7
- net /Display/~{BlkDispBuf}: track 0.00 -> 290.0 mm, vias 0 -> 7
- net Net-(U1-Pad1): track 0.00 -> 289.4 mm, vias 0 -> 7
- net Net-(U1-Pad2): track 0.00 -> 279.7 mm, vias 0 -> 4
- net Net-(U1-Pad5): track 0.00 -> 111.9 mm, vias 0 -> 4
- net +3.3V: track 0.00 -> 102.4 mm, vias 0 -> 1
- net Net-(U12-Pad5): track 0.00 -> 97.0 mm, vias 0 -> 1
- net Net-(U11-Pad5): track 0.00 -> 92.0 mm, vias 0 -> 1
- net Net-(U3-Pad5): track 0.00 -> 67.7 mm, vias 0 -> 4
- net Net-(U6-Pad10): track 0.00 -> 64.8 mm, vias 0 -> 2
- net ~{BlkDisp}: track 0.00 -> 61.7 mm, vias 0 -> 2
- net DispC: track 0.00 -> 60.0 mm, vias 0 -> 2
- net DispB: track 0.00 -> 50.5 mm, vias 0 -> 2
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
Commit message: WIP: PCB design
Parts:
- C1, C10, C11, C12, C13, C14, C16, C17, C2, C3, C4, C5, C6, C7, C8, C9: footprint Capacitor_THT:C_Disc_D5.0mm_W2.5mm_P5.00mm -> Capacitor_SMD:C_1206_3216Metric_Pad1.33x1.80mm_HandSolder
- C19, C22: footprint Capacitor_THT:C_Disc_D6.0mm_W2.5mm_P5.00mm -> Capacitor_SMD:C_1206_3216Metric_Pad1.33x1.80mm_HandSolder
- R53, R58: moved to B.Cu
- moved C26 512.0 mm to (72.6, 138.4), turned to 180 degrees
- moved C27 494.3 mm to (110.4, 105.0), turned to 180 degrees
- moved C21 487.4 mm to (71.4, 116.7), turned to 180 degrees
- moved C20 484.3 mm to (71.4, 126.7), turned to 180 degrees
- moved C23 483.9 mm to (85.8, 105.0), turned to 180 degrees
- moved R58 461.4 mm to (71.9, 107.2), turned to 180 degrees
- moved R53 455.1 mm to (71.9, 102.6), turned to 180 degrees
- moved C24 454.8 mm to (94.1, 105.0), turned to 180 degrees
- moved J2 441.3 mm to (65.8, 148.8), turned to 180 degrees
- moved J1 429.2 mm to (74.0, 148.8), turned to 180 degrees
- moved C22 406.9 mm to (118.0, 108.7)
- moved C2 404.1 mm to (114.0, 89.6), turned to -90 degrees
- moved C12 370.2 mm to (142.3, 125.6), turned to -90 degrees
- moved C25 342.8 mm to (210.5, 108.2), turned to 90 degrees
- moved C18 339.8 mm to (200.9, 108.2), turned to 90 degrees
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Connections:
- U4 pad 10: Net-(R38-Pad1) -> Net-(R35-Pad1)
- U4 pad 11: Net-(R35-Pad1) -> Net-(R38-Pad1)
Routing:
- net /Display/LedsGnd: track 0.00 -> 378.5 mm, vias 0 -> 5
- net +3.3V: track 102.4 -> 325.3 mm, vias 1 -> 8
- net +12V: track 421.0 -> 630.3 mm
- net +5V: track 0.00 -> 157.7 mm
- net Net-(R15-Pad1): track 0.00 -> 140.3 mm, vias 0 -> 1
- net Net-(R18-Pad1): track 0.00 -> 112.3 mm, vias 0 -> 1
- net Net-(U10-Pad10): track 0.00 -> 104.5 mm, vias 0 -> 2
- net Net-(U10-Pad11): track 0.00 -> 99.0 mm, vias 0 -> 2
- net DispD: track 48.4 -> 133.6 mm, vias 2 -> 3
- net Net-(U10-Pad2): track 0.00 -> 84.8 mm, vias 0 -> 2
- net Net-(U12-Pad5): track 97.0 -> 177.9 mm, vias 1 -> 2
- net DispB: track 50.5 -> 130.2 mm, vias 2 -> 3
- net Net-(U10-Pad1): track 0.00 -> 76.6 mm, vias 0 -> 2
- net DispA: track 50.1 -> 126.0 mm
- net DispSel2: track 0.00 -> 74.7 mm, vias 0 -> 2
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Other:
- board outline added: 336.1 x 75.3 mm

Commit message: Better routing
Parts:
- moved C17 27.7 mm to (213.6, 107.0)
- moved C22 10.4 mm to (108.1, 111.9), turned to 180 degrees
- moved C19 7.04 mm to (111.6, 144.0), turned to 90 degrees
- moved C16 5.90 mm to (213.6, 115.6)
- moved C15 1.55 mm to (209.0, 116.8)
- moved C25 1.55 mm to (209.0, 108.2)
Routing:
- net +3.3V: track 325.3 -> 427.0 mm, vias 8 -> 3
- net +12V: track 630.3 -> 649.1 mm, vias 10 -> 9
- net Net-(U1-Pad2): track 279.7 -> 295.9 mm, vias 4 -> 7
- net DispA: track 126.0 -> 135.8 mm
- net /Display/~{BlkDispBuf}: track 314.5 -> 322.9 mm
- net DispC: track 130.6 -> 138.2 mm
- net DispB: track 130.2 -> 137.2 mm
- net DispD: track 133.6 -> 139.5 mm
- net Net-(U1-Pad6): track 306.5 -> 311.8 mm
- net Net-(U1-Pad7): track 306.1 -> 309.6 mm
- net Net-(U3-Pad5): track 67.7 -> 64.9 mm, vias 4 -> 2
- net Net-(U10-Pad10): track 104.5 -> 101.9 mm
- net Net-(U1-Pad5): track 111.9 -> 109.5 mm, vias 4 -> 2
- net Net-(U5-Pad5): track 15.2 -> 17.5 mm
- net GND: track 2.00 -> 0.00 mm
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
Commit message: Ground fill and DRC fixes
Parts:
- moved R62 0.36 mm to (248.6, 83.0)
Routing:
- net +3.3V: track 427.0 -> 469.7 mm, vias 3 -> 4
- net +5V: track 158.8 -> 161.9 mm
- net DispD: track 139.5 -> 136.4 mm
- net +12V: track 649.1 -> 646.4 mm
- net DispB: track 137.2 -> 139.0 mm
- net Net-(U3-Pad5): track 64.9 -> 63.8 mm
- net Net-(R15-Pad1): track 140.3 -> 141.4 mm
- net ~{BlkDisp}: track 60.5 -> 59.4 mm
- net Net-(U6-Pad11): track 55.1 -> 56.1 mm
- net Net-(U5-Pad5): track 17.5 -> 16.7 mm
- net DispC: track 138.2 -> 137.4 mm
- net Net-(R4-Pad1): track 15.9 -> 15.2 mm
- net GND: vias 0 -> 37
- added copper zone on B.Cu, net GND
- added copper zone on F.Cu, net GND
Other:
- board size 336.1 x 75.3 mm -> 337 x 76.1 mm

Commit message: Finishing PCB design
Other:
- board text added: "12V"
- board text added: "GND"
